Commit message: i should've been updating this

File: assets/shelf/shelf.urdf (robot description, URDF)
Before this commit: robot shelf, 6 links, 5 joints
Links:
- removed link shelf_base
- removed link shelf_side1
- removed link shelf_side2
- removed link shelf_side3
- removed link shelf_side4
- added link back; collision box size=1.25 1.25 0.025; visual box size=1.25 1.25 0.025
- added link bottom; collision box size=0.3 1.25 0.025; visual box size=0.3 1.25 0.025
- added link left; collision box size=0.3 1.25 0.025; visual box size=0.3 1.25 0.025
- added link right; collision box size=0.3 1.25 0.025; visual box size=0.3 1.25 0.025
- added link top; collision box size=0.3 1.25 0.025; visual box size=0.3 1.25 0.025
Joints:
- removed joint shelf_joint1
- removed joint shelf_joint2
- removed joint shelf_joint3
- removed joint shelf_joint4
- added joint bottom_joint: type fixed, parent back, child bottom, origin xyz=0.6125  0 0.15 rpy=0 1.5708 0 
- added joint left_joint: type fixed, parent back, child left, origin xyz=0 -0.6125 0.15 rpy=1.5708 1.5708 0 
- added joint right_joint: type fixed, parent back, child right, origin xyz=0 0.6125 0.15 rpy=1.5708 1.5708 0 
- added joint top_joint: type fixed, parent back, child top, origin xyz=-0.6125 0 0.15 rpy=0 1.5708 0 
- joint center_base_joint: child shelf_base -> back; origin xyz=0 0 -0.25 rpy=0 0 0  -> xyz=0 0 -0.15 rpy=0 1.5708 0
